File: hardware/usb.sch (KiCad schematic (older format))
At the start: 2 parts

Commit message: update,
Connections:
- wire segments 24 -> 25
- no-connect marks 0 -> 1
Other:
- note added: "ESD OPTIONAL"
- moved on the sheet: U?
Changed lines of the file:
@@
 EESchema Schematic File Version 4
-LIBS:AMS1117-cache
+LIBS:STM32F042FxPx_tryout-cache
 EELAYER 29 0
 EELAYER END
-$Descr A4 11693 8268
+$Descr User 8500 5500
 encoding utf-8
 Sheet 3 3
@@
 L taobao-components:USB_Micro U?
 U 1 1 5D0E47F3
-P 2750 2150
-F 0 "U?" H 2750 2650 50  0000 C CNN
-F 1 "USB_Micro" H 2750 2550 50  0000 C CNN
-F 2 "footprint-lib:USB_Micro-B_Molex-105017-0001" H 2750 1650 50  0001 C CNN
-F 3 "" H 2750 1650 50  0001 C CNN
-	1    2750 2150
+P 1700 2150
+F 0 "U?" H 1700 2650 50  0000 C CNN
+F 1 "USB_Micro" H 1700 2550 50  0000 C CNN
+F 2 "footprint-lib:USB_Micro-B_Molex-105017-0001" H 1700 1650 50  0001 C CNN
+F 3 "" H 1700 1650 50  0001 C CNN
+	1    1700 2150
 	-1   0    0    -1
 $EndComp
@@
 L power:GND #PWR?
 U 1 1 5D0E4D6E
-P 2150 2650
-F 0 "#PWR?" H 2150 2400 50  0001 C CNN
-F 1 "GND" H 2200 2450 50  0000 C CNN
-F 2 "" H 2150 2650 50  0001 C CNN
-F 3 "" H 2150 2650 50  0001 C CNN
-	1    2150 2650
+P 1100 2650
+F 0 "#PWR?" H 1100 2400 50  0001 C CNN
+F 1 "GND" H 1150 2450 50  0000 C CNN
+F 2 "" H 1100 2650 50  0001 C CNN
+F 3 "" H 1100 2650 50  0001 C CNN
+	1    1100 2650
 	1    0    0    -1
 $EndComp
 Wire Wire Line
-	2150 2650 2150 2250
+	1100 2650 1100 2350
 Wire Wire Line
-	2150 1950 2350 1950
+	1100 1950 1300 1950
 Wire Wire Line
-	2350 2050 2150 2050
-Connection ~ 2150 2050
+	1300 2050 1100 2050
+Connection ~ 1100 2050
 Wire Wire Line
-	2150 2050 2150 1950
+	1100 2050 1100 1950
 Wire Wire Line
-	2150 2250 2350 2250
-Connection ~ 2150 2250
+	1100 2250 1300 2250
+Connection ~ 1100 2250
 Wire Wire Line
-	2150 2250 2150 2050
+	1100 2250 1100 2050
 Wire Wire Line
-	2150 2350 2350 2350
+	1100 2350 1300 2350
 $Comp
 L power:VBUS #PWR?
 U 1 1 5D0E5271
-P 3700 1700
-F 0 "#PWR?" H 3700 1550 50  0001 C CNN
-F 1 "VBUS" H 3750 1900 50  0000 C CNN
-F 2 "" H 3700 1700 50  0001 C CNN
-F 3 "" H 3700 1700 50  0001 C CNN
-	1    3700 1700
+P 3700 1150
+F 0 "#PWR?" H 3700 1000 50  0001 C CNN
+F 1 "VBUS" H 3750 1350 50  0000 C CNN
+F 2 "" H 3700 1150 50  0001 C CNN
+F 3 "" H 3700 1150 50  0001 C CNN
+	1    3700 1150
 	1    0    0    -1
 $EndComp
 Wire Wire Line
-	3700 1700 3700 1950
+	3700 1150 3700 1950
 Wire Wire Line
-	3700 1950 3150 1950
+	3700 1950 2100 1950
 $Comp
 L taobao-components:SRV05-4 U?
@@
 	1    0    0    -1
 $EndComp
-Text Label 4850 2050 2    50   ~ 0
+Text Label 6050 2050 2    50   ~ 0
 USB_N
-Text Label 4850 2150 2    50   ~ 0
+Text Label 6050 2150 2    50   ~ 0
 USB_P
 Wire Wire Line
-	3150 2050 4400 2050
+	2100 2050 4400 2050
 Wire Wire Line
-	3150 2150 3400 2150
+	2100 2150 3400 2150
 $Comp
 L power:GND #PWR?
 U 1 1 5D0EE2C4
-P 3250 2500
-F 0 "#PWR?" H 3250 2250 50  0001 C CNN
-F 1 "GND" H 3300 2300 50  0000 C CNN
-F 2 "" H 3250 2500 50  0001 C CNN
-F 3 "" H 3250 2500 50  0001 C CNN
-	1    3250 2500
+P 2350 2500
+F 0 "#PWR?" H 2350 2250 50  0001 C CNN
+F 1 "GND" H 2400 2300 50  0000 C CNN
+F 2 "" H 2350 2500 50  0001 C CNN
+F 3 "" H 2350 2500 50  0001 C CNN
+	1    2350 2500
 	1    0    0    -1
 $EndComp
 Wire Wire Line
-	3250 2500 3250 2350
+	2350 2500 2350 2350
 Wire Wire Line
-	3250 2350 3150 2350
+	2350 2350 2100 2350
 $Comp
 L power:GND #PWR?
@@
 Connection ~ 4400 2050
 Wire Wire Line
-	4400 2050 4850 2050
+	4400 2050 6050 2050
 Wire Wire Line
 	3450 2800 3400 2800
@@
 Connection ~ 3400 2150
 Wire Wire Line
-	3400 2150 4850 2150
+	3400 2150 6050 2150
+Connection ~ 1100 2350
+Wire Wire Line
+	1100 2350 1100 2250
+Wire Notes Line
+	3000 2500 3000 3500
+Wire Notes Line
+	3000 3500 4900 3500
+Wire Notes Line
+	4900 3500 4900 2500
+Wire Notes Line
+	4900 2500 3000 2500
+Text Notes 4850 3450 2    50   ~ 0
+ESD OPTIONAL
+NoConn ~ 2100 2250
 $EndSCHEMATC
